File: Projects/DMX-Adapter-small-V3/DMX-Adapter-small-V3.kicad_pcb (KiCad board)
At the start: 2 copper layers, 70 x 23 mm, 38 parts, among them J1 USB_B_Micro, J2 USART, J3 SWD, J4 DMX, Q2 2N7002, SW1 RST, SW2 BOOT0, U1 STM32F103C8T6, U2 SN75176BDR, U3 LM1117-3.3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

Commit message: preliminary final version
Parts:
- Q2: value 2N7002 -> Si2342DS
Changed lines of the file:
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@@
 			)
 		)
-		(property "Datasheet" "https://www.mouser.de/ProductDetail/KEMET/C0402C103K7PACTU?qs=DPoM0jnrROVPiEOKt2qSGA%3D%3D"
+		(property "Datasheet" "https://www.mouser.de/ProductDetail/Walsin/0402B103K6R3CT?qs=u16ybLDytRYFwOvCY%252Bt3gA%3D%3D"
 			(at 0 0 180)
 			(unlocked yes)
@@
 			)
 		)
-		(property "Mouser-Nr" "80-C0402C103K7PACTU"
+		(property "Mouser-Nr" "791-0402B103K6R3CT"
 			(at 0 0 180)
 			(unlocked yes)
@@
 			)
 		)
-		(property "Datasheet" "https://www.mouser.de/ProductDetail/KEMET/C0402C103K7PACTU?qs=DPoM0jnrROVPiEOKt2qSGA%3D%3D"
+		(property "Datasheet" "https://www.mouser.de/ProductDetail/Walsin/0402B103K6R3CT?qs=u16ybLDytRYFwOvCY%252Bt3gA%3D%3D"
 			(at 0 0 0)
 			(unlocked yes)
@@
 			)
 		)
-		(property "Mouser-Nr" "80-C0402C103K7PACTU"
+		(property "Mouser-Nr" "791-0402B103K6R3CT"
 			(at 0 0 0)
 			(unlocked yes)
@@
 			)
 		)
-		(property "Value" "2N7002"
+		(property "Value" "Si2342DS"
 			(at 0 -2.4 90)
 			(layer "B.Fab")
@@
 			)
 		)
-		(property "Datasheet" "https://www.mouser.de/ProductDetail/onsemi-Fairchild/NDS7002A?qs=HK%252BeIG1iaaix42XP2ZTlFA%3D%3D"
+		(property "Datasheet" "https://eu.mouser.com/ProductDetail/Vishay-Siliconix/SI2342DS-T1-GE3?qs=ROh%252BA47s9d0EG8kV%2FqrJ2w%3D%3D"
 			(at 0 0 90)
 			(layer "B.Fab")
@@
 			)
 		)
-		(property "Mouser-Nr" "512-NDS7002A"
+		(property "Mouser-Nr" "78-SI2342DS-T1-GE3"
 			(at 0 0 270)
 			(unlocked yes)
@@
 			)
 		)
-		(property "Datasheet" "https://www.mouser.de/ProductDetail/KEMET/C0402C103K7PACTU?qs=DPoM0jnrROVPiEOKt2qSGA%3D%3D"
+		(property "Datasheet" "https://www.mouser.de/ProductDetail/Walsin/0402B103K6R3CT?qs=u16ybLDytRYFwOvCY%252Bt3gA%3D%3D"
 			(at 0 0 180)
 			(unlocked yes)
@@
 			)
 		)
-		(property "Mouser-Nr" "80-C0402C103K7PACTU"
+		(property "Mouser-Nr" "791-0402B103K6R3CT"
 			(at 0 0 180)
 			(unlocked yes)
@@
 			)
 		)
-		(property "Datasheet" "https://www.mouser.de/ProductDetail/KEMET/C0402C103K7PACTU?qs=DPoM0jnrROVPiEOKt2qSGA%3D%3D"
+		(property "Datasheet" "https://www.mouser.de/ProductDetail/Walsin/0402B103K6R3CT?qs=u16ybLDytRYFwOvCY%252Bt3gA%3D%3D"
 			(at 0 0 270)
 			(unlocked yes)
@@
 			)
 		)
-		(property "Mouser-Nr" "80-C0402C103K7PACTU"
+		(property "Mouser-Nr" "791-0402B103K6R3CT"
 			(at 0 0 270)
 			(unlocked yes)
@@
 			)
 		)
-		(property "Datasheet" "https://www.mouser.de/ProductDetail/KEMET/C0402C103K7PACTU?qs=DPoM0jnrROVPiEOKt2qSGA%3D%3D"
+		(property "Datasheet" "https://www.mouser.de/ProductDetail/Walsin/0402B103K6R3CT?qs=u16ybLDytRYFwOvCY%252Bt3gA%3D%3D"
 			(at 0 0 90)
 			(unlocked yes)
@@
 			)
 		)
-		(property "Mouser-Nr" "80-C0402C103K7PACTU"
+		(property "Mouser-Nr" "791-0402B103K6R3CT"
 			(at 0 0 90)
 			(unlocked yes)

Commit message: final
Parts:
- added C14: 1u5, Capacitor_SMD:C_0603_1608Metric, B.Cu at (177.1, 44.7)
- added D2: GP, Diode_SMD:D_0603_1608Metric, F.Cu at (174.3, 41.0)
- added R5: 330R, Resistor_SMD:R_0402_1005Metric, B.Cu at (177.5, 40.0)
- added R7: 150R, Resistor_SMD:R_0402_1005Metric, F.Cu at (173.5, 45.2)
- added TP1: TX, TestPoint:TestPoint_Pad_D1.0mm, B.Cu at (162.2, 32.5)
- added TP2: DMX, TestPoint:TestPoint_Pad_D1.0mm, B.Cu at (160.8, 34.1)
- added TP3: INT, TestPoint:TestPoint_Pad_D1.0mm, B.Cu at (160.8, 38.1)
- C1, C2, C3, C4, C5: value 10n -> 100n
- Q2: value Si2342DS -> 2N7002
- R3: value 1k5 -> 330R
- moved R4 0.10 mm to (173.4, 46.4)
Connections:
- SW1 pad 2: NRST -> Net-(R7-Pad1)
- U1 pad 13: unconnected-(U1-PA3-Pad13) -> STAT_LED
Routing:
- net STAT_LED: track 0.00 -> 2.90 mm, vias 0 -> 1
- net Net-(Q2-D): track 3.52 -> 6.36 mm
- net Net-(D2-A): track 0.00 -> 2.37 mm, vias 0 -> 1
- net NRST: track 13.0 -> 14.9 mm
- net Net-(Q2-G): track 1.47 -> 3.12 mm
- net GND: track 32.5 -> 33.8 mm, vias 17 -> 18
- net Net-(R7-Pad1): track 0.00 -> 1.20 mm
