File: Projects/DMX-Adapter-small-V3/dmx_circuit.kicad_sch (KiCad schematic)
At the start: 5 parts, among them Q2 2N7002, U2 SN75176BDR

Commit message: preliminary final version
Parts:
- Q2: value 2N7002 -> Si2342DS
Changed lines of the file:
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@@
 	(polyline
 		(pts
-			(xy 101.6 40.64) (xy 57.15 40.64)
+			(xy 102.87 40.64) (xy 57.15 40.64)
 		)
 		(stroke
@@
 	(polyline
 		(pts
-			(xy 101.6 77.47) (xy 101.6 40.64)
+			(xy 102.87 77.47) (xy 102.87 40.64)
 		)
 		(stroke
@@
 	(polyline
 		(pts
-			(xy 57.15 77.47) (xy 101.6 77.47)
+			(xy 57.15 77.47) (xy 102.87 77.47)
 		)
 		(stroke
@@
 			)
 		)
-		(property "Value" "2N7002"
+		(property "Value" "Si2342DS"
 			(at 92.71 63.5 0)
 			(effects

Commit message: final
Parts:
- added TP1: TX, TestPoint:TestPoint_Pad_D1.0mm, symbol Connector:TestPoint
- added TP2: DMX, TestPoint:TestPoint_Pad_D1.0mm, symbol Connector:TestPoint
- added TP3: INT, TestPoint:TestPoint_Pad_D1.0mm, symbol Connector:TestPoint
- Q2: value Si2342DS -> 2N7002; Mouser-Nr 78-SI2342DS-T1-GE3 -> 512-2N7002
Connections:
- net USART_TX_DMX: now also TP1.1
- net at Q2.3 (D), R2.2, U2.4 (D): now also TP2.1
- net at Q2.1 (G), R8.2: now also TP3.1
