File: Projects/DMX-Adapter-small-V3/mcu.kicad_sch (KiCad schematic)
At the start: 11 parts, among them U1 STM32F103C8T6, Y1 Crystal_16MHz

Commit message: final
Parts:
- added D2: GP, Diode_SMD:D_0603_1608Metric, symbol Device:LED
- added R5: 330R, Resistor_SMD:R_0402_1005Metric, symbol Device:R
- C1, C2, C3, C4, C5: value 10n -> 100n; Mouser-Nr 791-0402B103K6R3CT -> 81-GRM152D70G104ME5D
- C6: Mouser-Nr 81-GRM188C80G226ME0D -> 81-GRM188C80J226ME5D
Connections:
- net GND: now also D2.1 (K)
- net STAT_LED: now reaches U1.13 (PA3)
- net STAT_LED: now also R5.1
- new net: D2.2 (A), R5.2
- no-connect marks 27 -> 26
Other:
- note added: "Status LED circuit"
- moved on the sheet: C8, C9, Y1
