File: Projects/DMX-Adapter-small-V3/power.kicad_sch (KiCad schematic)
At the start: 7 parts, among them U3 LM1117-3.3

Commit message: final
Parts:
- C12, C13: Mouser-Nr 81-GRM188C80G226ME0D -> 81-GRM188C80J226ME5D
- R3: value 1k5 -> 330R; Mouser-Nr 667-ERA-2VEB1501X -> 71-CRCW0402330RFKEDH
Changed lines of the file:
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@@
 			)
 		)
-		(property "Value" "1k5"
+		(property "Value" "330R"
 			(at 138.43 57.1499 0)
 			(effects
@@
 			)
 		)
-		(property "Datasheet" "https://www.mouser.de/ProductDetail/Panasonic/ERA-2VEB1501X?qs=OlC7AqGiEDkx8XOEQaRGXQ%3D%3D"
+		(property "Datasheet" "https://www.mouser.de/ProductDetail/Vishay-Dale/CRCW0402330RFKEDHP?qs=sGAEpiMZZMtlubZbdhIBIKMpMWeJoXcV1tfZ%252B52JmGI%3D"
 			(at 135.89 55.88 0)
 			(effects
@@
 			)
 		)
-		(property "Mouser-Nr" "667-ERA-2VEB1501X"
+		(property "Mouser-Nr" "71-CRCW0402330RFKEDH"
 			(at 135.89 55.88 0)
 			(effects
@@
 			)
 		)
-		(property "Datasheet" "https://www.mouser.de/ProductDetail/Murata-Electronics/GRM188C80G226MEA0D?qs=6V0hbkDBlKZLUx8AgMnILg%3D%3D"
+		(property "Datasheet" "https://www.mouser.de/ProductDetail/Murata-Electronics/GRM188C80J226ME15D?qs=K0Sa7bCb58I9yTIvpI1jlg%3D%3D"
 			(at 59.69 59.69 0)
 			(effects
@@
 			)
 		)
-		(property "Mouser-Nr" "81-GRM188C80G226ME0D"
+		(property "Mouser-Nr" "81-GRM188C80J226ME5D"
 			(at 59.69 59.69 0)
 			(effects
@@
 			)
 		)
-		(property "Datasheet" "https://www.mouser.de/ProductDetail/Murata-Electronics/GRM188C80G226MEA0D?qs=6V0hbkDBlKZLUx8AgMnILg%3D%3D"
+		(property "Datasheet" "https://www.mouser.de/ProductDetail/Murata-Electronics/GRM188C80J226ME15D?qs=K0Sa7bCb58I9yTIvpI1jlg%3D%3D"
 			(at 52.07 59.69 0)
 			(effects
@@
 			)
 		)
-		(property "Mouser-Nr" "81-GRM188C80G226ME0D"
+		(property "Mouser-Nr" "81-GRM188C80J226ME5D"
 			(at 52.07 59.69 0)
 			(effects
